File: ambient_light-cad/mcu.sch (KiCad schematic (older format))
At the start: 31 parts

Commit message: [Updated] move interface page and global label
interface 페이지에 들어가는 부품 이동 및 페이지 간 라벨링을 위해 Global label로 변경
Parts:
- removed C? (x4): 220μF, symbol Device:CP1_Small
- removed C?: 4.7μF, symbol Device:CP1_Small
- removed J?: ICSP, symbol Connector_Generic:Conn_02x03_Odd_Even
- removed J?: LED_Strip_conn_1, symbol Connector:Conn_01x03_Female
- removed J?: LED_Strip_conn_2, symbol Connector:Conn_01x03_Female
- removed J?: USB_C_Receptacle_USB2.0, symbol Connector:USB_C_Receptacle_USB2.0
Connections:
- net labels removed: VBUS
- wire segments 137 -> 96
- no-connect marks 10 -> 6
Other:
- moved on the sheet: D?
