File: ambient_light-cad/ambient_light-cad.sch (KiCad schematic (older format))
At the start: 0 parts

Commit message: [Modified] sync file
Changed lines of the file:
@@
 F0 "mcu" 50
 F1 "mcu.sch" 50
+$EndSheet
+$Sheet
 S 1950 3800 1750 1150
 U 5FDBFA91
